File: shift_led_driver.kicad_sch (KiCad schematic)
At the start: 6 parts, among them J10 Conn_02x05_Odd_Even, J11 Conn_02x05_Odd_Even, U4 TLC59282DBQR...SM16206

Commit message: use only rounded pads
Parts:
- U4: footprint Package_SO:QSOP-24_3.9x8.7mm_P0.635mm -> _my:QSOP-24_3.9x8.7mm_P0.635mm_rounded_pads
Changed lines of the file:
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@@
       (effects (font (size 1.27 1.27)) (justify left))
     )
-    (property "Footprint" "Package_SO:QSOP-24_3.9x8.7mm_P0.635mm" (id 2) (at 72.39 17.78 0)
+    (property "Footprint" "_my:QSOP-24_3.9x8.7mm_P0.635mm_rounded_pads" (id 2) (at 72.39 17.78 0)
       (effects (font (size 1.27 1.27)) hide)
     )
